Commit message: Edited LiDAR position

File: urdf/lidar.xacro (robot description, xacro)
@@ -4,5 +4,5 @@
         <parent link="frame" />
         <child link="laser_frame" />
-        <origin xyz="0 0 ${wheel_radius}" rpy="0 0 0" />
+        <origin xyz="0 0 ${wheel_radius+0.01}" rpy="0 0 0" />
     </joint>
     <link name="laser_frame">
