Commit message: Added another joint

File: urdf/ros2_control.xacro (robot description, xacro)
@@ -6,16 +6,18 @@
         </hardware>
         <joint name="steering_joint">
-            <command_interface name="position">
-                <param name="min">-1.570796327</param>
-                <param name="max">+1.570796327</param>
-            </command_interface>
+            <command_interface name="position" />
+            <command_interface name="velocity" />
             <state_interface name="position" />
             <state_interface name="velocity" />
         </joint>
         <joint name="traction_joint">
-            <command_interface name="velocity">
-                <param name="min">-1.0</param>
-                <param name="max">+1.0</param>
-            </command_interface>
+            <command_interface name="position" />
+            <command_interface name="velocity" />
+            <state_interface name="position" />
+            <state_interface name="velocity" />
+        </joint>
+        <joint name="front_traction_joint">
+            <command_interface name="position" />
+            <command_interface name="velocity" />
             <state_interface name="position" />
             <state_interface name="velocity" />
