Commit message: Thickened wheels

File: urdf/properties.xacro (robot description, xacro)
@@ -2,5 +2,5 @@
 <robot name="bicycle_drive" xmlns:xacro="http://ros.org/wiki/xacro">
     <xacro:property name="wheel_radius" value="0.25" />
-    <xacro:property name="wheel_thickness" value="0.1" />
+    <xacro:property name="wheel_thickness" value="0.2" />
     <xacro:property name="wheel_separation" value="0.98" />
     <xacro:property name="wheel_mass" value="1.0" />

Commit message: Added box length and mass

File: urdf/properties.xacro (robot description, xacro)
@@ -1,4 +1,6 @@
 <?xml version="1.0"?>
 <robot name="bicycle_drive" xmlns:xacro="http://ros.org/wiki/xacro">
+    <xacro:property name="box_length" value="0.01" />
+    <xacro:property name="box_mass" value="0.005" />
     <xacro:property name="wheel_radius" value="0.25" />
     <xacro:property name="wheel_thickness" value="0.2" />

Commit message: Removed unused properties

File: urdf/properties.xacro (robot description, xacro)
@@ -7,14 +7,5 @@
     <xacro:property name="wheel_separation" value="0.98" />
     <xacro:property name="wheel_mass" value="1.0" />
-    <xacro:property name="support_leg_mass" value="0.3" />
-    <xacro:property name="support_axis_mass" value="0.1" />
-    <xacro:property name="support_wheel_mass" value="0.5" />
-    <xacro:property name="frame_offset_z" value="${2*wheel_radius+const_1}" />
     <xacro:property name="frame_mass" value="1.5" />
-    <xacro:property name="screw_mass" value="0.2" />
-    <xacro:property name="seat_stay_mass" value="0.5" />
-    <xacro:property name="fork_mass" value="0.5" />
-    <xacro:property name="head_tube_mass" value="0.2" />
-    <xacro:property name="const_1" value="0.10" />
     <xacro:property name="cylindar_radius" value="0.01" />
 </robot>
