Commit message: Added wheels

File: urdf/bicycle_drive.xacro.urdf (robot description, URDF)
Before this commit: robot bicycle_drive, 3 links, 2 joints
Links:
- added link back_wheel; collision sphere radius=${wheel_radius}; visual cylinder length=${wheel_thickness} radius=${wheel_radius}
- added link front_wheel; collision sphere radius=${wheel_radius}; visual cylinder length=${wheel_thickness} radius=${wheel_radius}
Joints:
- added joint steering_joint: type continuous, parent frame, child front_wheel, origin xyz=0 ${wheel_separation/2} 0 rpy=0 ${pi/2} 0, axis 1 0 0
- added joint traction_joint: type continuous, parent frame, child back_wheel, origin xyz=0 ${-wheel_separation/2} 0 rpy=0 ${pi/2} 0, axis 0 0 1
- joint base_frame_joint: origin xyz=0 0 ${frame_offset_z} rpy=0 0 0 -> xyz=0 0 ${wheel_radius} rpy=0 0 0

Commit message: Flipped wheel orientation

File: urdf/bicycle_drive.xacro.urdf (robot description, URDF)
Before this commit: robot bicycle_drive, 5 links, 4 joints
Joints:
- joint traction_joint: origin xyz=0 ${-wheel_separation/2} 0 rpy=0 ${pi/2} 0 -> xyz=0 ${-wheel_separation/2} 0 rpy=0 ${-pi/2} 0

Commit message: Edited wheels collision

File: urdf/bicycle_drive.xacro.urdf (robot description, URDF)
Before this commit: robot bicycle_drive, 5 links, 4 joints
Links:
- link back_wheel: geometry collision cylinder length=${wheel_thickness} radius=${wheel_radius}; visual cylinder length=${wheel_thickness} radius=${wheel_radius}
- link front_wheel: geometry collision cylinder length=${wheel_thickness} radius=${wheel_radius}; visual cylinder length=${wheel_thickness} radius=${wheel_radius}

Commit message: Added steering_link

File: urdf/bicycle_drive.xacro.urdf (robot description, URDF)
Before this commit: robot bicycle_drive, 5 links, 4 joints
Links:
- added link steering_link; collision box size=${box_length} ${box_length} ${box_length}; visual box size=${box_length} ${box_length} ${box_length}
Joints:
- added joint front_traction_joint: type continuous, parent steering_link, child front_wheel, origin xyz=0 0 0 rpy=0 ${-pi/2} 0, axis 0 0 1
- joint steering_joint: axis 1 0 0 -> 0 0 1; child front_wheel -> steering_link; origin xyz=0 ${wheel_separation/2} 0 rpy=0 ${pi/2} 0 -> xyz=0 ${wheel_separation/2} 0 rpy=0 0 0

Commit message: Added mimic for front_traction_joint

File: urdf/bicycle_drive.xacro.urdf (robot description, URDF)
Before this commit: robot bicycle_drive, 6 links, 5 joints
Joints:
- joint front_traction_joint: mimic (none) -> joint=traction_joint

File: urdf/ros2_control.xacro (robot description, xacro)
@@ -22,6 +22,8 @@
         </joint>
         <joint name="front_traction_joint">
-            <!-- <param name="mimic">traction_joint</param> -->
-            <!-- <param name="multiplier">1</param> -->
+            <param name="mimic">traction_joint</param>
+            <param name="multiplier">1</param>
+            <command_interface name="position" />
+            <command_interface name="velocity" />
             <state_interface name="position" />
             <state_interface name="velocity" />

Commit message: Rotated base_link -90 deg

File: urdf/bicycle_drive.xacro.urdf (robot description, URDF)
Before this commit: robot bicycle_drive, 6 links, 5 joints
Joints:
- joint base_frame_joint: origin xyz=0 0 ${wheel_radius} rpy=0 0 0 -> xyz=0 0 ${wheel_radius} rpy=0 0 -${pi/2}
