Commit message: feat(description): simulator-independent bicycle description for Jazzy
New bicycle_description package. Fixes in the robot model:

- Frames follow REP-103/105: base_footprint is the root (it was a child
  of base_link) and sits under the rear axle, the reference point of the
  bicycle kinematics and of the steering controller's odometry (base_link
  used to be at the frame centre, half a wheelbase off).
- The model is built along +X; the -pi/2 yaw on the frame is gone.
- steering_joint is revolute with URDF limits (it was continuous and the
  limits only lived in ros2_control params, which Gazebo does not enforce).
- The front wheel is passive with state interfaces only, instead of
  mimicking the traction joint with the removed <param name="mimic">.
- Lidar: gpu_lidar for Gazebo Harmonic, gz_frame_id, <topic>scan, the
  <resoluation> typo fixed, 1 deg beams without a duplicated last beam,
  and a mast so the scan plane clears the wheel tops.
- Gazebo Classic material tags removed; realistic steering fork mass
  (was 5 g / 1 cm, a physics instability risk); wheel macro instead of
  copy-pasted wheel blocks.
- All dimensions come from config/geometry.yaml (single source of truth,
  loaded with xacro.load_yaml).
- The ros2_control hardware plugin is a xacro argument (Gazebo, mock or
  real hardware) and the gz_ros2_control plugin is only emitted with
  use_sim, so the hardware package can reuse this description.

Launch: description.launch.py (robot_state_publisher with
ParameterValue(Command(xacro)) and a real use_sim_time argument) and
display.launch.py (joint sliders + RViz, with a committed RViz config).

Tests: check_urdf, tree root, axle placement, joint types/limits, lidar,
ros2_control interfaces, hardware plugin selection.

Co-Authored-By: Claude Opus 5.5 <noreply@anthropic.com>

File: bicycle_description/urdf/bicycle.urdf.xacro (robot description, xacro)
@@ -1,52 +1,82 @@
 <?xml version="1.0"?>
-<robot name="bicycle_drive" xmlns:xacro="http://ros.org/wiki/xacro">
-    <!-- XACRO INCLUDE -->
+<!--
+  Self-driving bicycle. Frames follow REP-103/REP-105 (x forward, y left, z up).
+  base_footprint is the ground point under the rear axle: the reference point of the
+  bicycle kinematic model and of the bicycle_steering_controller odometry.
+  All dimensions come from config/geometry.yaml.
+  Arguments:
+    use_sim           "true" adds the Gazebo (gz_ros2_control) system plugin
+    hardware_plugin   ros2_control system plugin; empty selects GazeboSimSystem when
+                      use_sim is true, otherwise mock_components/GenericSystem
+    controllers_file  controller parameter file loaded by gz_ros2_control (use_sim only)
+-->
+<robot name="bicycle" xmlns:xacro="http://www.ros.org/wiki/xacro">
+    <xacro:arg name="use_sim" default="false" />
+    <xacro:arg name="hardware_plugin" default="" />
+    <xacro:arg name="controllers_file" default="" />
+    <xacro:include filename="inertial.xacro" />
     <xacro:include filename="materials.xacro" />
-    <xacro:include filename="properties.xacro" />
-    <xacro:include filename="inertial.xacro" />
+    <xacro:include filename="wheel.xacro" />
     <xacro:include filename="lidar.xacro" />
-    <!-- BASE LINK -->
+    <xacro:include filename="ros2_control.xacro" />
+    <xacro:property name="use_sim" value="${'$(arg use_sim)'.lower() in ('true', '1')}" />
+    <xacro:property name="geometry"
+        value="${xacro.load_yaml('$(find bicycle_description)/config/geometry.yaml')}" />
+    <xacro:property name="wheelbase" value="${geometry.wheelbase}" />
+    <xacro:property name="wheel" value="${geometry.wheel}" />
+    <xacro:property name="chassis" value="${geometry.chassis}" />
+    <xacro:property name="steering" value="${geometry.steering}" />
+    <xacro:property name="traction" value="${geometry.traction}" />
+    <!-- BASE -->
+    <link name="base_footprint" />
+    <joint name="base_joint" type="fixed">
+        <parent link="base_footprint" />
+        <child link="base_link" />
+        <origin xyz="0 0 ${wheel.radius}" rpy="0 0 0" />
+    </joint>
+    <!-- Rear axle centre. -->
     <link name="base_link" />
-    <!-- BASE FOOTPRINT LINK -->
-    <joint name="base_footprint_joint" type="fixed">
+    <!-- CHASSIS: frame tube between the two axles -->
+    <joint name="chassis_joint" type="fixed">
         <parent link="base_link" />
-        <child link="base_footprint" />
-        <origin xyz="0 0 0" rpy="0 0 0" />
+        <child link="chassis" />
+        <origin xyz="${wheelbase/2} 0 0" rpy="0 0 0" />
     </joint>
-    <link name="base_footprint" />
-    <!-- FRAME LINK -->
-    <joint name="base_frame_joint" type="fixed">
-        <parent link="base_link" />
-        <child link="frame" />
-        <origin xyz="0 0 ${wheel_radius}" rpy="0 0 -${pi/2}" />
-    </joint>
-    <link name="frame">
+    <link name="chassis">
         <visual>
-            <origin xyz="0 0 0" rpy="${pi/2} 0 0" />
+            <origin xyz="0 0 0" rpy="0 ${pi/2} 0" />
             <geometry>
-                <cylinder length="${wheel_separation}" radius="${cylindar_radius}" />
+                <cylinder length="${wheelbase}" radius="${chassis.tube_radius}" />
             </geometry>
             <material name="cyan" />
         </visual>
         <collision>
-            <origin xyz="0 0 0" rpy="${pi/2} 0 0" />
+            <origin xyz="0 0 0" rpy="0 ${pi/2} 0" />
             <geometry>
-                <cylinder length="${wheel_separation}" radius="${cylindar_radius}" />
+                <cylinder length="${wheelbase}" radius="${chassis.tube_radius}" />
             </geometry>
         </collision>
-        <xacro:inertial_cylinder mass="${frame_mass}" length="${wheel_separation}"
-            radius="${cylindar_radius}">
-            <origin xyz="0 0 0" rpy="${pi/2} 0 0" />
+        <xacro:inertial_cylinder mass="${chassis.mass}" length="${wheelbase}"
+            radius="${chassis.tube_radius}">
+            <origin xyz="0 0 0" rpy="0 ${pi/2} 0" />
         </xacro:inertial_cylinder>
     </link>
-    <gazebo reference="frame">
-        <material>Gazebo/Turquoise</material>
-    </gazebo>
-    <!-- STEERING LINK -->
-    <joint name="steering_joint" type="continuous">
+    <!-- REAR (TRACTION) WHEEL -->
+    <joint name="traction_joint" type="continuous">
+        <parent link="base_link" />
+        <child link="rear_wheel" />
+        <origin xyz="0 0 0" rpy="0 0 0" />
+        <axis xyz="0 1 0" />
+        <limit effort="${traction.max_effort}" velocity="${traction.max_velocity}" />
+    </joint>
+    <xacro:wheel_link name="rear_wheel" config="${wheel}" />
+    <!-- STEERING FORK at the front axle -->
+    <joint name="steering_joint" type="revolute">
+        <parent link="base_link" />
+        <child link="steering_link" />
+        <origin xyz="${wheelbase} 0 0" rpy="0 0 0" />
         <axis xyz="0 0 1" />
-        <parent link="frame" />
-        <child link="steering_link" />
-        <origin xyz="0 ${wheel_separation/2} 0" rpy="0 0 0" />
+        <limit lower="${-steering.max_angle}" upper="${steering.max_angle}"
+            effort="${steering.max_effort}" velocity="${steering.max_velocity}" />
     </joint>
     <link name="steering_link">
@@ -54,5 +84,5 @@
             <origin xyz="0 0 0" rpy="0 0 0" />
             <geometry>
-                <box size="${box_length} ${box_length} ${box_length}" />
+                <box size="${steering.fork_size} ${steering.fork_size} ${steering.fork_size}" />
             </geometry>
             <material name="white" />
@@ -61,78 +91,29 @@
             <origin xyz="0 0 0" rpy="0 0 0" />
             <geometry>
-                <box size="${box_length} ${box_length} ${box_length}" />
+                <box size="${steering.fork_size} ${steering.fork_size} ${steering.fork_size}" />
             </geometry>
         </collision>
-        <xacro:inertial_box mass="${box_mass}"
-            x="${box_length}" y="${box_length}" z="${box_length}">
+        <xacro:inertial_box mass="${steering.fork_mass}"
+            x="${steering.fork_size}" y="${steering.fork_size}" z="${steering.fork_size}">
             <origin xyz="0 0 0" rpy="0 0 0" />
         </xacro:inertial_box>
     </link>
-    <gazebo reference="steering_link">
-        <material>Gazebo/White</material>
-    </gazebo>
-    <!-- FRONT WHEEL -->
-    <joint name="front_traction_joint" type="continuous">
-        <mimic joint="traction_joint" />
-        <axis xyz="0 0 1" />
+    <!-- FRONT WHEEL (passive) -->
+    <joint name="front_wheel_joint" type="continuous">
         <parent link="steering_link" />
         <child link="front_wheel" />
-        <origin xyz="0 0 0" rpy="0 ${-pi/2} 0" />
+        <origin xyz="0 0 0" rpy="0 0 0" />
+        <axis xyz="0 1 0" />
     </joint>
-    <link name="front_wheel">
-        <visual>
-            <origin xyz="0 0 0" rpy="0 0 0" />
-            <geometry>
-                <cylinder length="${wheel_thickness}" radius="${wheel_radius}" />
-            </geometry>
-            <material name="black" />
-        </visual>
-        <collision>
-            <origin xyz="0 0 0" rpy="0 0 0" />
-            <geometry>
-                <cylinder length="${wheel_thickness}" radius="${wheel_radius}" />
-            </geometry>
-        </collision>
-        <xacro:inertial_cylinder mass="${wheel_mass}" length="${wheel_thickness}"
-            radius="${wheel_radius}">
-            <origin xyz="0 0 0" rpy="0 0 0" />
-        </xacro:inertial_cylinder>
-    </link>
-    <gazebo reference="front_wheel">
-        <material>Gazebo/Black</material>
-        <mu1 value="0.5" />
-        <mu2 value="0.5" />
-    </gazebo>
-    <!-- BACK OR TRACTION WHEEL -->
-    <joint name="traction_joint" type="continuous">
-        <axis xyz="0 0 1" />
-        <parent link="frame" />
-        <child link="back_wheel" />
-        <origin xyz="0 ${-wheel_separation/2} 0" rpy="0 ${-pi/2} 0" />
-    </joint>
-    <link name="back_wheel">
-        <visual>
-            <origin xyz="0 0 0" rpy="0 0 0" />
-            <geometry>
-                <cylinder length="${wheel_thickness}" radius="${wheel_radius}" />
-            </geometry>
-            <material name="black" />
-        </visual>
-        <collision>
-            <origin xyz="0 0 0" rpy="0 0 0" />
-            <geometry>
-                <cylinder length="${wheel_thickness}" radius="${wheel_radius}" />
-            </geometry>
-        </collision>
-        <xacro:inertial_cylinder mass="${wheel_mass}" length="${wheel_thickness}"
-            radius="${wheel_radius}">
-            <origin xyz="0 0 0" rpy="0 0 0" />
-        </xacro:inertial_cylinder>
-    </link>
-    <gazebo reference="back_wheel">
-        <material>Gazebo/Black</material>
-        <!-- <mu1 value="0.5" /> -->
-        <!-- <mu2 value="0.5" /> -->
-    </gazebo>
-    <xacro:include filename="ros2_control.xacro" />
+    <xacro:wheel_link name="front_wheel" config="${wheel}" />
+    <!-- SENSORS -->
+    <xacro:lidar parent="chassis" mount_z="${geometry.lidar.scan_height - wheel.radius}"
+        config="${geometry.lidar}" />
+    <!-- ROS2 CONTROL -->
+    <xacro:property name="default_hardware_plugin"
+        value="${'gz_ros2_control/GazeboSimSystem' if use_sim else 'mock_components/GenericSystem'}" />
+    <xacro:bicycle_ros2_control
+        hardware_plugin="${'$(arg hardware_plugin)' or default_hardware_plugin}"
+        use_sim="${use_sim}"
+        controllers_file="$(arg controllers_file)" />
 </robot>

File: bicycle_description/urdf/inertial.xacro (robot description, xacro)
@@ -1,4 +1,5 @@
 <?xml version="1.0"?>
-<robot name="bicycle_drive" xmlns:xacro="http://ros.org/wiki/xacro">
+<robot xmlns:xacro="http://www.ros.org/wiki/xacro">
+    <!-- Solid cylinder whose axis is the z axis of the given origin. -->
     <xacro:macro name="inertial_cylinder" params="mass length radius *origin">
         <inertial>
@@ -11,4 +12,5 @@
         </inertial>
     </xacro:macro>
+    <!-- Solid box with edges x, y, z along the axes of the given origin. -->
     <xacro:macro name="inertial_box" params="mass x y z *origin">
         <inertial>

File: bicycle_description/urdf/lidar.xacro (robot description, xacro)
@@ -1,55 +1,74 @@
 <?xml version="1.0"?>
-<robot name="bicycle_drive" xmlns:xacro="http://ros.org/wiki/xacro">
-    <joint name="frame_lidar" type="fixed">
-        <parent link="frame" />
-        <child link="laser_frame" />
-        <origin xyz="0 0 ${wheel_radius+0.01}" rpy="0 0 0" />
-    </joint>
-    <link name="laser_frame">
-        <visual>
-            <origin xyz="0 0 0" rpy="0 0 0" />
-            <geometry>
-                <cylinder length="0.01" radius="0.07" />
-            </geometry>
-            <material name="black" />
-        </visual>
-        <collision>
-            <geometry>
-                <cylinder length="0.01" radius="0.07" />
-            </geometry>
-        </collision>
-        <xacro:inertial_cylinder mass="0.5" length="0.01" radius="0.07">
-            <origin xyz="0 0 0" rpy="0 0 0" />
-        </xacro:inertial_cylinder>
-    </link>
-    <gazebo reference="laser_frame">
-        <sensor name="laser" type="ray">
-            <pose>0 0 0 0 0 0</pose>
-            <visualize>true</visualize>
-            <update_rate>9</update_rate>
-            <ray>
-                <scan>
-                    <horizontal>
-                        <samples>360</samples>
-                        <resoluation>1</resoluation>
-                        <min_angle>-3.14</min_angle>
-                        <max_angle>3.14</max_angle>
-                    </horizontal>
-                </scan>
-                <range>
-                    <min>0.12</min>
-                    <max>10.0</max>
-                    <resoluation>0.01</resoluation>
-                </range>
-            </ray>
-            <plugin name="laser_controller" filename="libgazebo_ros_ray_sensor.so">
-                <ros>
-                    <argument>--ros-args --remap ~/out:=scan</argument>
-                </ros>
-                <output_type>sensor_msgs/LaserScan</output_type>
-                <frame_name>laser_frame</frame_name>
-            </plugin>
-        </sensor>
-        <material>Gazebo/Black</material>
-    </gazebo>
+<robot xmlns:xacro="http://www.ros.org/wiki/xacro">
+    <!--
+      2D lidar on a mast. The sensor publishes sensor_msgs/LaserScan on /scan
+      (bridged from Gazebo) in frame laser_frame.
+      parent:  link the mast stands on
+      mount_z: height of the scan plane above the parent link origin [m]
+      config:  the `lidar` block of config/geometry.yaml
+    -->
+    <xacro:macro name="lidar" params="parent mount_z config">
+        <xacro:property name="mast_length" value="${mount_z - config.length/2}" />
+        <joint name="laser_joint" type="fixed">
+            <parent link="${parent}" />
+            <child link="laser_frame" />
+            <origin xyz="0 0 ${mount_z}" rpy="0 0 0" />
+        </joint>
+        <link name="laser_frame">
+            <visual>
+                <origin xyz="0 0 0" rpy="0 0 0" />
+                <geometry>
+                    <cylinder length="${config.length}" radius="${config.radius}" />
+                </geometry>
+                <material name="black" />
+            </visual>
+            <visual>
+                <origin xyz="0 0 ${-(mount_z + config.length/2)/2}" rpy="0 0 0" />
+                <geometry>
+                    <cylinder length="${mast_length}" radius="${config.mast_radius}" />
+                </geometry>
+                <material name="black" />
+            </visual>
+            <collision>
+                <origin xyz="0 0 0" rpy="0 0 0" />
+                <geometry>
+                    <cylinder length="${config.length}" radius="${config.radius}" />
+                </geometry>
+            </collision>
+            <xacro:inertial_cylinder mass="${config.mass}" length="${config.length}"
+                radius="${config.radius}">
+                <origin xyz="0 0 0" rpy="0 0 0" />
+            </xacro:inertial_cylinder>
+        </link>
+        <gazebo reference="laser_frame">
+            <sensor name="lidar" type="gpu_lidar">
+                <topic>scan</topic>
+                <gz_frame_id>laser_frame</gz_frame_id>
+                <always_on>true</always_on>
+                <visualize>true</visualize>
+                <update_rate>${config.update_rate}</update_rate>
+                <lidar>
+                    <scan>
+                        <horizontal>
+                            <samples>${config.samples}</samples>
+                            <resolution>1</resolution>
+                            <!-- Full circle without a duplicated first/last beam. -->
+                            <min_angle>${-pi}</min_angle>
+                            <max_angle>${pi - 2*pi/config.samples}</max_angle>
+                        </horizontal>
+                    </scan>
+                    <range>
+                        <min>${config.min_range}</min>
+                        <max>${config.max_range}</max>
+                        <resolution>0.01</resolution>
+                    </range>
+                    <noise>
+                        <type>gaussian</type>
+                        <mean>0.0</mean>
+                        <stddev>0.01</stddev>
+                    </noise>
+                </lidar>
+            </sensor>
+        </gazebo>
+    </xacro:macro>
 </robot>

File: bicycle_description/urdf/materials.xacro (robot description, xacro)
@@ -1,4 +1,4 @@
 <?xml version="1.0"?>
-<robot name="bicycle_drive" xmlns:xacro="http://ros.org/wiki/xacro">
+<robot xmlns:xacro="http://www.ros.org/wiki/xacro">
     <material name="white">
         <color rgba="1 1 1 1" />
@@ -7,12 +7,6 @@
         <color rgba="0.18 0.83 0.78 1" />
     </material>
-    <material name="blue">
-        <color rgba="0.2 0.2 1 1" />
-    </material>
     <material name="black">
-        <color rgba="0 0 0 1" />
-    </material>
-    <material name="red">
-        <color rgba="1 0 0 1" />
+        <color rgba="0.05 0.05 0.05 1" />
     </material>
 </robot>

File: bicycle_description/urdf/ros2_control.xacro (robot description, xacro)
@@ -1,44 +1,42 @@
 <?xml version="1.0"?>
-<robot name="bicycle_drive" xmlns:xacro="http://ros.org/wiki/xacro">
-    <ros2_control name="GazeboSystem" type="system">
-        <hardware>
-            <plugin>gazebo_ros2_control/GazeboSystem</plugin>
-        </hardware>
-        <joint name="steering_joint">
-            <command_interface name="position">
-                <param name="min">-0.7854</param>
-                <param name="max">+0.7854</param>
-            </command_interface>
-            <state_interface name="position" />
-            <state_interface name="velocity" />
-        </joint>
-        <joint name="traction_joint">
-            <command_interface name="velocity">
-                <param name="min">-1.0</param>
-                <param name="max">+1.0</param>
-            </command_interface>
-            <state_interface name="position" />
-            <state_interface name="velocity" />
-        </joint>
-        <joint name="front_traction_joint">
-            <param name="mimic">traction_joint</param>
-            <param name="multiplier">1</param>
-            <command_interface name="position" />
-            <command_interface name="velocity" />
-            <state_interface name="position" />
-            <state_interface name="velocity" />
-        </joint>
-    </ros2_control>
-    <gazebo>
-        <plugin name="gazebo_ros2_control" filename="libgazebo_ros2_control.so">
-            <parameters>
-                $(find self_driving_bicycle)/config/bicycle_drive_controller.yaml
-            </parameters>
-            <ros>
-                <remapping>
-                    /bicycle_controller/tf_odometry:=/tf
-                </remapping>
-            </ros>
-        </plugin>
-    </gazebo>
+<robot xmlns:xacro="http://www.ros.org/wiki/xacro">
+    <!--
+      ros2_control system of the bicycle. The hardware plugin is injected so the same
+      description serves Gazebo, mock hardware (tests) and the real robot.
+      hardware_plugin:  ros2_control SystemInterface plugin name
+      use_sim:          add the gz_ros2_control Gazebo system plugin
+      controllers_file: controller parameter file loaded by gz_ros2_control (use_sim only)
+    -->
+    <xacro:macro name="bicycle_ros2_control" params="hardware_plugin use_sim controllers_file">
+        <ros2_control name="BicycleSystem" type="system">
+            <hardware>
+                <plugin>${hardware_plugin}</plugin>
+            </hardware>
+            <!-- Front-wheel steering: position command. -->
+            <joint name="steering_joint">
+                <command_interface name="position" />
+                <state_interface name="position" />
+                <state_interface name="velocity" />
+            </joint>
+            <!-- Rear-wheel drive: velocity command. -->
+            <joint name="traction_joint">
+                <command_interface name="velocity" />
+                <state_interface name="position" />
+                <state_interface name="velocity" />
+            </joint>
+            <!-- Passive front wheel: state only, so its TF is still published. -->
+            <joint name="front_wheel_joint">
+                <state_interface name="position" />
+                <state_interface name="velocity" />
+            </joint>
+        </ros2_control>
+        <xacro:if value="${use_sim}">
+            <gazebo>
+                <plugin filename="gz_ros2_control-system"
+                    name="gz_ros2_control::GazeboSimROS2ControlPlugin">
+                    <parameters>${controllers_file}</parameters>
+                </plugin>
+            </gazebo>
+        </xacro:if>
+    </xacro:macro>
 </robot>
