Commit message: feat(description): hardware parameters from a YAML file
New xacro and launch argument hardware_params_file: every key of the
flat YAML file becomes a <param> of the ros2_control <hardware> block.
The real robot passes bicycle_hardware/config/hardware.yaml, so the
description stays free of hardware details and the hardware package no
longer needs its own copy of the URDF.

Co-Authored-By: Claude Opus 5.5 <noreply@anthropic.com>

File: bicycle_description/urdf/bicycle.urdf.xacro (robot description, xacro)
@@ -9,4 +9,7 @@
     hardware_plugin   ros2_control system plugin; empty selects GazeboSimSystem when
                       use_sim is true, otherwise mock_components/GenericSystem
+    hardware_params_file
+                      YAML file of the plugin's hardware parameters (flat key: value);
+                      empty for none
     controllers_file  controller parameter file loaded by gz_ros2_control (use_sim only)
 -->
@@ -14,4 +17,5 @@
     <xacro:arg name="use_sim" default="false" />
     <xacro:arg name="hardware_plugin" default="" />
+    <xacro:arg name="hardware_params_file" default="" />
     <xacro:arg name="controllers_file" default="" />
     <xacro:include filename="inertial.xacro" />
@@ -113,6 +117,8 @@
     <xacro:property name="default_hardware_plugin"
         value="${'gz_ros2_control/GazeboSimSystem' if use_sim else 'mock_components/GenericSystem'}" />
+    <xacro:property name="hardware_params_file" value="$(arg hardware_params_file)" />
     <xacro:bicycle_ros2_control
         hardware_plugin="${'$(arg hardware_plugin)' or default_hardware_plugin}"
+        hardware_params="${list(xacro.load_yaml(hardware_params_file).items()) if hardware_params_file else []}"
         use_sim="${use_sim}"
         controllers_file="$(arg controllers_file)" />

File: bicycle_description/urdf/ros2_control.xacro (robot description, xacro)
@@ -1,15 +1,25 @@
 <?xml version="1.0"?>
 <robot xmlns:xacro="http://www.ros.org/wiki/xacro">
+    <!-- One <param name="key">value</param> per (key, value) pair of `params`. -->
+    <xacro:macro name="hardware_params" params="params">
+        <xacro:if value="${params}">
+            <param name="${params[0][0]}">${params[0][1]}</param>
+            <xacro:hardware_params params="${params[1:]}" />
+        </xacro:if>
+    </xacro:macro>
     <!--
       ros2_control system of the bicycle. The hardware plugin is injected so the same
       description serves Gazebo, mock hardware (tests) and the real robot.
       hardware_plugin:  ros2_control SystemInterface plugin name
+      hardware_params:  list of (name, value) hardware parameters of the plugin
       use_sim:          add the gz_ros2_control Gazebo system plugin
       controllers_file: controller parameter file loaded by gz_ros2_control (use_sim only)
     -->
-    <xacro:macro name="bicycle_ros2_control" params="hardware_plugin use_sim controllers_file">
+    <xacro:macro name="bicycle_ros2_control"
+        params="hardware_plugin hardware_params use_sim controllers_file">
         <ros2_control name="BicycleSystem" type="system">
             <hardware>
                 <plugin>${hardware_plugin}</plugin>
+                <xacro:hardware_params params="${hardware_params}" />
             </hardware>
             <!-- Front-wheel steering: position command. -->
